File: RGB_LED_matrix_PCB/RGB_LED_matrix_PCB.kicad_pcb (KiCad board)
At the start: 2 copper layers, 200 parts, among them U1 WS2815F, U10 WS2815F, U100 WS2815F, U11 WS2815F, U12 WS2815F, U13 WS2815F, U14 WS2815F, U15 WS2815F, U16 WS2815F, U17 WS2815F, U18 WS2815F, U19 WS2815F, U2 WS2815F, U20 WS2815F, U21 WS2815F, U22 WS2815F, U23 WS2815F, U24 WS2815F, U25 WS2815F, U26 WS2815F, U27 WS2815F, U28 WS2815F, U29 WS2815F, U3 WS2815F, U30 WS2815F, U31 WS2815F, U32 WS2815F, U33 WS2815F, U34 WS2815F, U35 WS2815F, U36 WS2815F, U37 WS2815F, U38 WS2815F, U39 WS2815F, U4 WS2815F, U40 WS2815F, U41 WS2815F, U42 WS2815F, U43 WS2815F, U44 WS2815F, U45 WS2815F, U46 WS2815F, U47 WS2815F, U48 WS2815F, U49 WS2815F, U5 WS2815F, U50 WS2815F, U51 WS2815F, U52 WS2815F, U53 WS2815F, U54 WS2815F, U55 WS2815F, U56 WS2815F, U57 WS2815F, U58 WS2815F, U59 WS2815F, U6 WS2815F, U60 WS2815F, U61 WS2815F, U62 WS2815F, U63 WS2815F, U64 WS2815F, U65 WS2815F, U66 WS2815F, U67 WS2815F, U68 WS2815F, U69 WS2815F, U7 WS2815F, U70 WS2815F, U71 WS2815F, U72 WS2815F, U73 WS2815F, U74 WS2815F, U75 WS2815F, U76 WS2815F, U77 WS2815F, U78 WS2815F, U79 WS2815F, U8 WS2815F, U80 WS2815F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

Commit message: Fixed some issues with the layout
Parts:
- moved C10 0.30 mm to (191.0, 51.6)
- moved C100 0.30 mm to (191.0, 141.6)
- moved C12 0.30 mm to (151.0, 61.6)
- moved C14 0.30 mm to (161.0, 61.6)
- moved C16 0.30 mm to (171.0, 61.6)
- moved C17 0.30 mm to (131.0, 61.6)
- moved C18 0.30 mm to (181.0, 61.6)
- moved C19 0.30 mm to (141.0, 61.6)
- moved C20 0.30 mm to (191.0, 61.6)
- moved C22 0.30 mm to (151.0, 71.6)
- moved C24 0.30 mm to (161.0, 71.6)
- moved C26 0.30 mm to (171.0, 71.6)
- moved C27 0.30 mm to (131.0, 71.6)
- moved C28 0.30 mm to (181.0, 71.6)
- moved C29 0.30 mm to (141.0, 71.6)
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Routing:
- net /LED_ROW5/DOUT2: track 115.5 -> 222.5 mm
- net +12V: track 658.5 -> 628.5 mm
- net /LED_ROW8/DOUT2: track 115.5 -> 113.8 mm
- net /LED_ROW6/DOUT2: track 115.5 -> 113.8 mm
- net /LED_ROW3/DOUT2: track 115.5 -> 113.8 mm
- net /LED_ROW1/DOUT2: track 115.5 -> 113.8 mm
- net /LED_ROW7/DOUT2: track 115.5 -> 113.8 mm
- net /LED_ROW4/DOUT2: track 115.5 -> 113.8 mm
- net /LED_ROW2/DOUT2: track 115.5 -> 113.8 mm
- net /LED_ROW/DOUT2: track 115.5 -> 113.8 mm
- net /LED_ROW8/DOUT1: track 219.4 -> 217.9 mm
- net /LED_ROW1/DOUT1: track 219.4 -> 217.9 mm
- net /LED_ROW7/DOUT1: track 219.4 -> 217.9 mm
- net /LED_ROW6/DOUT1: track 219.4 -> 217.9 mm
- net /LED_ROW5/DOUT1: track 219.4 -> 217.9 mm
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- added copper zone on B.Cu, net GND
- added copper zone on F.Cu, net GND
- removed copper zone on F.Cu, net unconnected-(U4-NC-Pad1)
