File: RGB_LED_matrix_PCB/RGB_LED_matrix_PCB.kicad_pcb (KiCad board)
At the start: 2 copper layers, 99.5 x 99.5 mm, 235 parts, among them CN1 B03B-XASK-1-A(LF)(SN), U1 WS2815F, U10 WS2815F, U100 WS2815F, U11 WS2815F, U12 WS2815F, U13 WS2815F, U14 WS2815F, U15 WS2815F, U16 WS2815F, U17 WS2815F, U18 WS2815F, U19 WS2815F, U2 WS2815F, U20 WS2815F, U21 WS2815F, U22 WS2815F, U23 WS2815F, U24 WS2815F, U25 WS2815F, U26 WS2815F, U27 WS2815F, U28 WS2815F, U29 WS2815F, U3 WS2815F, U30 WS2815F, U31 WS2815F, U32 WS2815F, U33 WS2815F, U34 WS2815F, U35 WS2815F, U36 WS2815F, U37 WS2815F, U38 WS2815F, U39 WS2815F, U4 WS2815F, U40 WS2815F, U41 WS2815F, U42 WS2815F, U43 WS2815F, U44 WS2815F, U45 WS2815F, U46 WS2815F, U47 WS2815F, U48 WS2815F, U49 WS2815F, U5 WS2815F, U50 WS2815F, U51 WS2815F, U52 WS2815F, U53 WS2815F, U54 WS2815F, U55 WS2815F, U56 WS2815F, U57 WS2815F, U58 WS2815F, U59 WS2815F, U6 WS2815F, U60 WS2815F, U61 WS2815F, U62 WS2815F, U63 WS2815F, U64 WS2815F, U65 WS2815F, U66 WS2815F, U67 WS2815F, U68 WS2815F, U69 WS2815F, U7 WS2815F, U70 WS2815F, U71 WS2815F, U72 WS2815F, U73 WS2815F, U74 WS2815F, U75 WS2815F, U76 WS2815F, U77 WS2815F, U78 WS2815F, U79 WS2815F, U8 WS2815F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

Commit message: Forgot to add the LED matrix pcb to the last commit, same thing as with the UPDCB.
Parts:
- added G***: LOGO, LOGO, B.Cu at (188.5, 132.1)
- added G***: LOGO, LOGO, B.Cu at (160.8, 127.2)
- added G***: LOGO, LOGO, B.Cu at (194.8, 114.6)
- added G***: LOGO, LOGO, B.Cu at (191.8, 109.9)
- added H1: MountingHole_Pad, MountingHole:MountingHole_2.2mm_M2_DIN965_Pad_TopOnly, B.Cu at (117.0, 127.0)
- added H2: MountingHole_Pad, MountingHole:MountingHole_2.2mm_M2_DIN965_Pad_TopOnly, B.Cu at (177.0, 127.0)
- added H3: MountingHole_Pad, MountingHole:MountingHole_2.2mm_M2_DIN965_Pad_TopOnly, B.Cu at (117.0, 67.0)
- added H4: MountingHole_Pad, MountingHole:MountingHole_2.2mm_M2_DIN965_Pad_TopOnly, B.Cu at (177.0, 67.0)
- added REF**: OSHW-Logo2_14.6x12mm_SilkScreen, Symbol:OSHW-Logo2_14.6x12mm_SilkScreen, B.Cu at (139.5, 135.0)
- added REF**: ESD-Logo_13.2x12mm_SilkScreen, Symbol:ESD-Logo_13.2x12mm_SilkScreen, B.Cu at (138.7, 120.2)
- added kobee-studio-6AA92370: Kobee Studio, kobee-studio-6AA92370, B.Cu at (193.8, 67.5)
- added kobee-studio-6AA9F6C4: Kobee Studio, kobee-studio-6AA9F6C4, B.Cu at (152.5, 127.2)
- added kobee-studio-6AA9F9DB: Kobee Studio, kobee-studio-6AA9F9DB, B.Cu at (145.3, 66.7)
Routing:
- net GND: vias 463 -> 459
