File: RGB_LED_matrix_PCB/10_LED_row/10_LED_row.kicad_pcb (KiCad board)
At the start: 2 copper layers, 20 parts, among them U1 WS2815F, U10 WS2815F, U2 WS2815F, U3 WS2815F, U4 WS2815F, U5 WS2815F, U6 WS2815F, U7 WS2815F, U8 WS2815F, U9 WS2815F

Commit message: Routed the matrix structure
Parts:
- moved C1 0.85 mm to (103.3, 99.6)
- moved C2 0.85 mm to (113.3, 99.6)
- moved C3 0.85 mm to (123.3, 99.6)
- moved C10 0.85 mm to (193.3, 99.6)
- moved C4 0.85 mm to (133.3, 99.6)
- moved C5 0.85 mm to (143.3, 99.6)
- moved C6 0.85 mm to (153.3, 99.6)
- moved C7 0.85 mm to (163.3, 99.6)
- moved C8 0.85 mm to (173.3, 99.6)
- moved C9 0.85 mm to (183.3, 99.6)
- moved U1 0.85 mm to (99.0, 99.0)
- moved U10 0.85 mm to (189.0, 99.0)
- moved U2 0.85 mm to (109.0, 99.0)
- moved U3 0.85 mm to (119.0, 99.0)
- moved U4 0.85 mm to (129.0, 99.0)
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Routing:
- net /DOUT1: track 0.00 -> 106.1 mm, vias 0 -> 2
- net /DOUT2: track 11.6 -> 113.9 mm

Commit message: Fixed some issues with the layout
Parts:
- moved C10 0.30 mm to (193.0, 99.6)
- moved C4 0.30 mm to (133.0, 99.6)
- moved C5 0.30 mm to (143.0, 99.6)
- moved C6 0.30 mm to (153.0, 99.6)
- moved C7 0.30 mm to (163.0, 99.6)
- moved C8 0.30 mm to (173.0, 99.6)
- moved C9 0.30 mm to (183.0, 99.6)
- moved C1 0.30 mm to (103.0, 99.6)
- moved C2 0.30 mm to (113.0, 99.6)
- moved C3 0.30 mm to (123.0, 99.6)
Routing:
- net +12V: track 65.9 -> 62.9 mm
- net /DOUT2: track 113.9 -> 112.2 mm
