File: RGB_LED_matrix_PCB/10_LED_row/10_LED_row.kicad_sch (KiCad schematic)
At the start: 20 parts, among them U1 WS2815F, U10 WS2815F, U2 WS2815F, U3 WS2815F, U4 WS2815F, U5 WS2815F, U6 WS2815F, U7 WS2815F, U8 WS2815F, U9 WS2815F

Commit message: Finished the LED matrix board layout - it just needs some polishing now and minor fixes
Other:
- title: (none) -> RGB LED MATRIX
Changed lines of the file:
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@@
 	(generator_version "10.0")
 	(paper "A4")
+	(title_block
+		(title "RGB LED MATRIX")
+		(rev "1.0")
+	)
 	(junction
 		(at 161.29 147.32)
