File: RGB_LED_matrix_PCB/PD_section/PD_section.kicad_sch (KiCad schematic)
At the start: 45 parts, among them Q1 AO4407A, Q2 AO4407A, Q3 AO3401A, U1 HUSB238A-xxxxx-QN16R, U2 TPS54202DDC

Commit message: Changed the USB connector to one that is compatible with higher PD voltages. Further proceeded with PD section routing
Parts:
- removed USB1, USB2: TYPE-C 16P QTWT, lcsc_footprints:C5187472_USB-TYPE-C-SMD_TYPE-C-16P-QTWT, symbol lcsc_imported:TYPE-C_16P_QTWT
- added USB1, USB2: TYPE-C 16P QTGM027, lcsc_footprints:C5187472_USB-TYPE-C-SMD_TYPE-C-16P-QTWT, symbol lcsc_imported:TYPE-C_16P_QTGM027_v2
Connections:
- net +5V_VSYS: now also Q3.3 (D); no longer Q3.2 (S)
- net D+: now also USB2.A6 (DP1), USB2.B6 (DP2)
- net D-: now also USB2.A7 (DN1), USB2.B7 (DN2)
- net GND: now also USB1.0 (EH), USB1.A1B12 (GND), USB1.B1A12 (GND), USB2.0 (EH), USB2.A1B12 (GND), USB2.B1A12 (GND)
- net IND_LED_DOUT: now also LED1.3 (DOUT); no longer LED2.3 (DOUT)
- net USB1_D+: now also USB1.A6 (DP1), USB1.B6 (DP2)
- net USB1_D-: now also USB1.A7 (DN1), USB1.B7 (DN2)
- net at C13.1, C2.1, C3.2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: now also USB1.A4B9 (VBUS), USB1.B4A9 (VBUS)
- net at U1.3 (CC1): now also USB1.A5 (CC1)
- net at U1.4 (CC2): now also USB1.B5 (CC2)
- net at LED1.1 (DIN): now also LED2.3 (DOUT); no longer R11.2
- net at F1.2: now also USB2.A4B9 (VBUS), USB2.B4A9 (VBUS)
- net at R5.1, R9.1: now also USB2.A5 (CC1)
- net at R10.1, R6.1: now also USB2.B5 (CC2)
- net at C6.2, C7.1, L1.2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: now also Q3.2 (S); no longer Q3.3 (D)
- net at LED2.1 (DIN): now also R11.2; no longer LED1.3 (DOUT)
Other:
- moved on the sheet: Q3
