File: RGB_LED_matrix_PCB/_restore_backup_2026-08-21T00-06-08-023/RGB_LED_matrix_PCB.kicad_pcb (KiCad board)
At the start: 2 copper layers, 100 x 100 mm, 215 parts, among them CN1 B03B-XASK-1-A(LF)(SN), U1 WS2815F, U10 WS2815F, U100 WS2815F, U11 WS2815F, U12 WS2815F, U13 WS2815F, U14 WS2815F, U15 WS2815F, U16 WS2815F, U17 WS2815F, U18 WS2815F, U19 WS2815F, U2 WS2815F, U20 WS2815F, U21 WS2815F, U22 WS2815F, U23 WS2815F, U24 WS2815F, U25 WS2815F, U26 WS2815F, U27 WS2815F, U28 WS2815F, U29 WS2815F, U3 WS2815F, U30 WS2815F, U31 WS2815F, U32 WS2815F, U33 WS2815F, U34 WS2815F, U35 WS2815F, U36 WS2815F, U37 WS2815F, U38 WS2815F, U39 WS2815F, U4 WS2815F, U40 WS2815F, U41 WS2815F, U42 WS2815F, U43 WS2815F, U44 WS2815F, U45 WS2815F, U46 WS2815F, U47 WS2815F, U48 WS2815F, U49 WS2815F, U5 WS2815F, U50 WS2815F, U51 WS2815F, U52 WS2815F, U53 WS2815F, U54 WS2815F, U55 WS2815F, U56 WS2815F, U57 WS2815F, U58 WS2815F, U59 WS2815F, U6 WS2815F, U60 WS2815F, U61 WS2815F, U62 WS2815F, U63 WS2815F, U64 WS2815F, U65 WS2815F, U66 WS2815F, U67 WS2815F, U68 WS2815F, U69 WS2815F, U7 WS2815F, U70 WS2815F, U71 WS2815F, U72 WS2815F, U73 WS2815F, U74 WS2815F, U75 WS2815F, U76 WS2815F, U77 WS2815F, U78 WS2815F, U79 WS2815F, U8 WS2815F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

Commit message: Changed LED matrix pcb design to a serpentine structure for better signal integrity. Proceeded with adding the connector and capacitors.
Parts:
- removed C101, C102, C103, C104, C105, C106, C107, C108, C109, C110: RZE-35V101MF80UQ-R2, lcsc_footprints:C19673858_CAP-SMD_BD6_3-L6_5-W6_5-LS7_2-FD_1
- removed CN1: B03B-XASK-1-A(LF)(SN), lcsc_footprints:C264992_CONN-TH_B03B-XASK-1-A-LF-SN
- removed R1: 470R, Resistor_SMD:R_0402_1005Metric_Pad0.72x0.64mm_HandSolder
- removed TP1: DOUT, TestPoint:TestPoint_Pad_D1.0mm
- removed TP2: DOUT_B, TestPoint:TestPoint_Pad_D1.0mm
- removed kibuzzard-6A877ACD: G***, kibuzzard-6A877ACD
Connections:
- U1 pad 6: GND -> /LED_ROW/DIN2
