File: Universal_Power_Delivery_and_Control_Board/TPS51385.kicad_sch (KiCad schematic)
At the start: 15 parts, among them U8 TPS51385RJNR

Commit message: Finally figured out the soft start circuitry.
Parts:
- added C27: 160nF, Capacitor_SMD:C_0402_1005Metric_Pad0.74x0.62mm_HandSolder, symbol Device:C
- added CN1, CN2, CN3, CN4: B03B-XASK-1-A(LF)(SN), lcsc_footprints:C264992_CONN-TH_B03B-XASK-1-A-LF-SN, symbol lcsc_imported:B03B-XASK-1-A(LF)(SN)
- added R16: 1K, Resistor_SMD:R_0402_1005Metric_Pad0.72x0.64mm_HandSolder, symbol Device:R
- added R17: 10K, Resistor_SMD:R_0402_1005Metric_Pad0.72x0.64mm_HandSolder, symbol Device:R
- added U9: TPS24751RUVR, lcsc_footprints:C2653596_VQFN-36_L7_0-W3_5-P0_50-BL-EP, symbol lcsc_imported:TPS24751RUVR
- C19: now fitted
Connections:
- net +12V_PD: now also U9.14 (DRAIN), U9.15 (DRAIN), U9.16 (DRIAN), U9.17 (DRAIN), U9.18 (DRAIN), U9.26 (SENSE), U9.27 (DRAIN), U9.29 (VCC), U9.3 (SET), U9.38 (DRAIN), U9.5 (DRAIN)
- net GND: now also CN1.3, CN2.3, CN3.3, CN4.3, R16.2, R17.2, U9.1 (OV), U9.2 (IMON), U9.28 (GND), U9.32 (GND), U9.34 (PROG), U9.35 (TIMER), U9.36 (GND), U9.37 (GND), U9.4 (GND)
- net VOUT renamed VOUT_connectors
- net VOUT_connectors: now also CN1.1, CN2.1, CN3.1, CN4.1, U9.10 (OUT), U9.11 (OUT), U9.12 (OUT), U9.13 (OUT), U9.19 (OUT), U9.20 (OUT), U9.21 (OUT), U9.22 (OUT), U9.23 (OUT), U9.24 (OUT), U9.6 (OUT), U9.7 (OUT), U9.8 (OUT), U9.9 (OUT)
- new net: C27.1, U9.25 (GATE)
- new net: C27.2, R16.1
- new net SOFT_START_EN: R17.1, U9.33 (EN)
- no-connect marks 1 -> 3
Other:
- note added: "Calculated for a 65ms raise time, while keeping the max inrush around 1.5~1.6A."
- moved on the sheet: C14, C15, C16, C17, C18, C20, C21, C22, C23, L2, R12, R13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
