File: Universal_Power_Delivery_and_Control_Board/UI_Section.kicad_sch (KiCad schematic)
At the start: 28 parts, among them SW2 TS1102-TD35HBM, SW3 TS1102-TD35HBM, SW4 TS1102-TD35HBM, U17 SN74LVC1G17DCKR, U23 SN74LVC1G17DCKR

Commit message: Finished layout 0 DRC errors.
Parts:
- added C56: 10uF, Capacitor_SMD:C_0805_2012Metric_Pad1.18x1.45mm_HandSolder, symbol Device:C
Connections:
- net +5V_VSYS: now also C56.2
- net GND: now also C56.1
Changed lines of the file:
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@@
 	)
 	(junction
+		(at 77.47 68.58)
+		(diameter 0)
+		(color 0 0 0 0)
+	)
+	(junction
 		(at 204.47 77.47)
 		(diameter 0)
@@
 	(wire
 		(pts
+			(xy 77.47 86.36) (xy 77.47 90.17)
+		)
+		(stroke
+			(width 0)
+			(type default)
+		)
+	)
+	(wire
+		(pts
 			(xy 168.91 83.82) (xy 171.45 83.82)
 		)
@@
 	(wire
 		(pts
+			(xy 77.47 68.58) (xy 77.47 78.74)
+		)
+		(stroke
+			(width 0)
+			(type default)
+		)
+	)
+	(wire
+		(pts
 			(xy 204.47 77.47) (xy 204.47 85.09)
 		)
@@
 	(wire
 		(pts
+			(xy 72.39 68.58) (xy 77.47 68.58)
+		)
+		(stroke
+			(width 0)
+			(type default)
+		)
+	)
+	(wire
+		(pts
 			(xy 158.75 73.66) (xy 158.75 83.82)
 		)
@@
 	(wire
 		(pts
-			(xy 72.39 60.96) (xy 72.39 68.58)
+			(xy 77.47 60.96) (xy 77.47 68.58)
 		)
 		(stroke
@@
 	(symbol
 		(lib_id "power:+1V0")
-		(at 72.39 60.96 0)
+		(at 77.47 60.96 0)
 		(unit 1)
 		(body_style 1)
@@
 		(fields_autoplaced yes)
 		(property "Reference" "#PWR069"
-			(at 72.39 64.77 0)
+			(at 77.47 64.77 0)
 			(hide yes)
 			(show_name no)
@@
 		)
 		(property "Value" "+5V_VSYS"
-			(at 72.39 55.88 0)
+			(at 77.47 55.88 0)
 			(show_name no)
 			(do_not_autoplace no)
@@
 		)
 		(property "Footprint" ""
-			(at 72.39 60.96 0)
+			(at 77.47 60.96 0)
 			(hide yes)
 			(show_name no)
@@
 		)
 		(property "Datasheet" ""
-			(at 72.39 60.96 0)
+			(at 77.47 60.96 0)
 			(hide yes)
 			(show_name no)
@@
 		)
 		(property "Description" "Power symbol creates a global label with name \"+1V0\""
-			(at 72.39 60.96 0)
+			(at 77.47 60.96 0)
 			(hide yes)
 			(show_name no)
@@
 	(symbol
 		(lib_id "power:GND")
+		(at 77.47 90.17 0)
+		(unit 1)
+		(body_style 1)
+		(exclude_from_sim no)
+		(in_bom yes)
+		(on_board yes)
+		(in_pos_files yes)
+		(dnp no)
+		(fields_autoplaced yes)
+		(property "Reference" "#PWR0107"
+			(at 77.47 96.52 0)
+			(hide yes)
+			(show_name no)
+			(do_not_autoplace no)
+			(effects
+				(font
+					(size 1.27 1.27)
+				)
+			)
+		)
+		(property "Value" "GND"
+			(at 77.47 95.25 0)
+			(show_name no)
+			(do_not_autoplace no)
+			(effects
+				(font
+					(size 1.27 1.27)
+				)
+			)
+		)
+		(property "Footprint" ""
+			(at 77.47 90.17 0)
+			(hide yes)
+			(show_name no)
+			(do_not_autoplace no)
+			(effects
+				(font
+					(size 1.27 1.27)
+				)
+			)
+		)
+		(property "Datasheet" ""
+			(at 77.47 90.17 0)
+			(hide yes)
+			(show_name no)
+			(do_not_autoplace no)
+			(effects
+				(font
+					(size 1.27 1.27)
+				)
+			)
+		)
+		(property "Description" "Power symbol creates a global label with name \"GND\" , ground"
+			(at 77.47 90.17 0)
+			(hide yes)
+			(show_name no)
+			(do_not_autoplace no)
+			(effects
+				(font
+					(size 1.27 1.27)
+				)
+			)
+		)
+		(pin "1"
+		)
+		(instances
+			(project "Universal_Power_Delivery_and_Control_Board"
+				(path "/b749dd2f-6b66-411b-a989-65da6091f700/1cd07b1f-498b-40ff-9a00-834575d9cc68"
+					(reference "#PWR0107")
+					(unit 1)
+				)
+			)
+		)
+	)
+	(symbol
+		(lib_id "power:GND")
 		(at 158.75 146.05 0)
 		(unit 1)
@@
 					(unit 1)
 				)
+			)
+		)
+	)
+	(symbol
+		(lib_id "Device:C")
+		(at 77.47 82.55 180)
+		(unit 1)
+		(body_style 1)
+		(exclude_from_sim no)
+		(in_bom yes)
+		(on_board yes)
+		(in_pos_files yes)
+		(dnp no)
+		(property "Reference" "C56"
+			(at 81.28 83.8201 0)
+			(show_name no)
+			(do_not_autoplace no)
+			(effects
+				(font
+					(size 1.27 1.27)
+				)
+				(justify right)
+			)
+		)
+		(property "Value" "10uF"
+			(at 81.28 81.2801 0)
+			(show_name no)
+			(do_not_autoplace no)
+			(effects
+				(font
+					(size 1.27 1.27)
+				)
+				(justify right)
+			)
+		)
+		(property "Footprint" "Capacitor_SMD:C_0805_2012Metric_Pad1.18x1.45mm_HandSolder"
+			(at 76.5048 78.74 0)
+			(hide yes)
+			(show_name no)
+			(do_not_autoplace no)
+			(effects
+				(font
+					(size 1.27 1.27)
+				)
+			)
+		)
+		(property "Datasheet" ""
+			(at 77.47 82.55 0)
+			(hide yes)
+			(show_name no)
+			(do_not_autoplace no)
+			(effects
+				(font
+					(size 1.27 1.27)
+				)
+			)
+		)
+		(property "Description" "Unpolarized capacitor"
+			(at 77.47 82.55 0)
+			(hide yes)
+			(show_name no)
+			(do_not_autoplace no)
+			(effects
+				(font
+					(size 1.27 1.27)
+				)
+			)
+		)
+		(pin "1"
+		)
+		(pin "2"
+		)
+		(instances
+			(project "Universal_Power_Delivery_and_Control_Board"
+				(path "/b749dd2f-6b66-411b-a989-65da6091f700/1cd07b1f-498b-40ff-9a00-834575d9cc68"
+					(reference "C56")
+					(unit 1)
+				)

Commit message: Small mostly cosmetic changes and reannotation of the schematic, followed by the export of the gerber files for production.
Parts:
- removed C36: 100nF, Capacitor_SMD:C_0402_1005Metric_Pad0.74x0.62mm_HandSolder, symbol Device:C
- removed C56: 10uF, Capacitor_SMD:C_0805_2012Metric_Pad1.18x1.45mm_HandSolder, symbol Device:C
- removed U17, U23: SN74LVC1G17DCKR, lcsc_footprints:C10425_SC-70-5_L2_1-W1_3-P0_65-LS2_1-BR, symbol lcsc_imported:SN74LVC1G17DCKR
- added C49: 100nF, Capacitor_SMD:C_0402_1005Metric_Pad0.74x0.62mm_HandSolder, symbol Device:C
- added C59: 10uF, Capacitor_SMD:C_0805_2012Metric_Pad1.18x1.45mm_HandSolder, symbol Device:C
- added U24, U25: SN74LV1T34DCK, Package_TO_SOT_SMD:SOT-353_SC-70-5, symbol Logic_LevelTranslator:SN74LV1T34DCK
- renumbered C35 to C50, C47 to C51, C48 to C52, C49 to C53, C50 to C54, C51 to C55, C52 to C56, C7 to C57, C5 to C58, LED3 to LED1, LED4 to LED2, LED5 to LED3, LED2 to LED4, LED1 to LED5, R39 to R42, R41 to R43, R43 to R44, R29 to R45, R40 to R46, R42 to R47, R44 to R48, R7 to R49
Connections:
- net +5V_VSYS: now also C49.1, C59.1, U24.5 (VCC), U25.5 (VCC)
- net Button_LED_DIN: now also U24.2 (A)
- net GND: now also C49.2, C59.2, U24.3 (GND), U25.3 (GND)
- net IND_LED_DIN: now also U25.2 (A)
- net at R49.1: now also U25.4 (Y)
- net at R45.1: now also U24.4 (Y)
- no-connect marks 4 -> 2
Other:
- note added: "replace with TI SN74LV1T34DCKR"
- company: (none) -> Jan Ścibielski
- title: (none) -> UI Section
- moved on the sheet: C56

Commit message: Added some design variants and and changed some componenets values within them. Added interactive HTML BOMs via plugin.
Other:
- note added: "NOTE (NOT APPLICABLE TO THE 5x5x5-LED-CUBE-SC IT MUST USE THE IC ON THE SCHEMATIC): Can be replaced with SN74LVC1G17DCKR and it should work although using the one on the schematic is preffered."
- note removed: "replace with TI SN74LV1T34DCKR"
Changed lines of the file:
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@@
 		(company "Jan Ścibielski")
 	)
-	(text "replace with TI SN74LV1T34DCKR\n"
+	(text "NOTE (NOT APPLICABLE TO THE 5x5x5-LED-CUBE-SC\nIT MUST USE THE IC ON THE SCHEMATIC):\nCan be replaced with SN74LVC1G17DCKR and it should work although\nusing the one on the schematic is preffered.\n"
 		(exclude_from_sim no)
-		(at 91.948 113.284 0)
+		(at 65.786 47.752 0)
 		(effects
 			(font
@@
 		)
 	)
+	(polyline
+		(pts
+			(xy 73.66 60.96) (xy 73.66 63.5)
+		)
+		(stroke
+			(width 0)
+			(type dash_dot_dot)
+			(color 255 155 1 1)
+		)
+	)
 	(wire
 		(pts
@@
 		)
 	)
+	(polyline
+		(pts
+			(xy 66.04 63.5) (xy 66.04 68.58)
+		)
+		(stroke
+			(width 0)
+			(type dash_dot_dot)
+			(color 255 155 1 1)
+		)
+	)
 	(wire
 		(pts
@@
 		)
 	)
+	(polyline
+		(pts
+			(xy 73.66 60.96) (xy 73.66 53.34)
+		)
+		(stroke
+			(width 0)
+			(type dash_dot_dot)
+			(color 255 155 1 1)
+		)
+	)
 	(wire
 		(pts
@@
 		)
 	)
+	(polyline
+		(pts
+			(xy 73.66 63.5) (xy 66.04 63.5)
+		)
+		(stroke
+			(width 0)
+			(type dash_dot_dot)
+			(color 255 155 1 1)
+		)
+	)
