File: Universal_Power_Delivery_and_Control_Board/Universal_Power_Delivery_and_Control_Board.kicad_sch (KiCad schematic)
At the start: 30 parts, among them Q1 JTD2302, SW1 TSA016A2526A, U1 SC7A20HTR, U2 S2B-ZR (LF)(SN), U3 TCA9555PWR, U4 HC-PM254-8.5H-2X4PW-02A, U5 TF-0803-0

Commit message: Added some design variants and and changed some componenets values within them. Added interactive HTML BOMs via plugin.
Parts:
- R3, R4: now fitted
Changed lines of the file:
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@@
 					(reference "R6")
 					(unit 1)
+					(variant
+						(name "10x10-LED-MATRIX")
+						(dnp yes)
+					)
+					(variant
+						(name "20x20-LED-MATRIX")
+						(dnp yes)
+					)
+					(variant
+						(name "5x5x5-LED-CUBE-RGB")
+						(dnp yes)
+					)
 				)
 			)
@@
 					(reference "R7")
 					(unit 1)
+					(variant
+						(name "10x10-LED-MATRIX")
+						(dnp yes)
+					)
+					(variant
+						(name "20x20-LED-MATRIX")
+						(dnp yes)
+					)
+					(variant
+						(name "5x5x5-LED-CUBE-RGB")
+						(dnp yes)
+					)
 				)
 			)
@@
 					(reference "R8")
 					(unit 1)
+					(variant
+						(name "10x10-LED-MATRIX")
+						(dnp yes)
+					)
+					(variant
+						(name "20x20-LED-MATRIX")
+						(dnp yes)
+					)
+					(variant
+						(name "5x5x5-LED-CUBE-RGB")
+						(dnp yes)
+					)
 				)
 			)
@@
 		(on_board yes)
 		(in_pos_files yes)
-		(dnp yes)
+		(dnp no)
 		(property "Reference" "R4"
 			(at 112.268 85.5979 0)
@@
 					(reference "R4")
 					(unit 1)
+					(variant
+						(name "10x10-LED-MATRIX")
+						(dnp yes)
+					)
+					(variant
+						(name "10x10x10-LED-CUBE-SC")
+						(dnp yes)
+					)
+					(variant
+						(name "20x20-LED-MATRIX")
+						(dnp yes)
+					)
+					(variant
+						(name "5x5x5-LED-CUBE-RGB")
+						(dnp yes)
+					)
 				)
 			)
@@
 		(on_board yes)
 		(in_pos_files yes)
-		(dnp yes)
+		(dnp no)
 		(property "Reference" "R3"
 			(at 102.362 87.8841 0)
@@
 					(reference "R3")
 					(unit 1)
+					(variant
+						(name "10x10-LED-MATRIX")
+						(dnp yes)
+					)
+					(variant
+						(name "10x10x10-LED-CUBE-SC")
+						(dnp yes)
+					)
+					(variant
+						(name "20x20-LED-MATRIX")
+						(dnp yes)
+					)
+					(variant
+						(name "5x5x5-LED-CUBE-RGB")
+						(dnp yes)
+					)
 				)
 			)
@@
 				(path "/b749dd2f-6b66-411b-a989-65da6091f700"
 					(page "4")
+					(variant
+						(name "10x10-LED-MATRIX")
+						(dnp yes)
+					)
+					(variant
+						(name "20x20-LED-MATRIX")
+						(dnp yes)
+					)
+					(variant
+						(name "5x5x5-LED-CUBE-RGB")
+						(dnp yes)
+					)
 				)
 			)
